File: Tello_Power_PCB.sch (EAGLE design)
At the start: 105 parts, among them CON1 XT30PW-F, CON2 XT30PW-F, CON3 XT30PW-F, CON4 XT30PW-F, CON7 XT60PW-M, J1 PJ-002A, J2 1719740002, J3 1719740002, J4 1719740002, J5 1719740002, J6 1719740002, J7 1719740002, J8 1719740002, J9 1719740002, M1 30V, M2 60V, M3 30V, M4 60V, Q1 BSC027N06LS5ATMA1, Q2 BSC027N06LS5ATMA1, Q3 IXTA96P085T, Q7 IXTA96P085T, Q8 IXTA96P085T, Q9 IXTA96P085T, U1 LM3150MH/NOPB, U11 TLV7041DCKR, U12 DMN67D8LW-13, U2 LM3150MH/NOPB, U3 LTC4357CMS8TRPBF, U4 ADS1015IDGSR, U5 MIC5282-3.3YMM-TR, U6 DMN67D8LW-13, U7 DMN67D8LW-13, U8 LTC4357CMS8TRPBF, U9 TLV6713DDCTDDC0006A_M

Commit message: added ADC and 5V-AO
Parts:
- removed U5: MIC5282-3.3YMM-TR, MIC5282-3-3YMM:MIC5282-3.3YMM-TR
- added C37: 2.2uF, rcl:C-EUC0603
- added C38: 2.2uF, rcl:C-EUC1206
- added C39: 10µF, microbuilder:CAP_CERAMIC0603
- added J10: SM02BGHSTBLFSN, SM02B-GHS-TB:SM02BGHSTBLFSN
- added JP1: (no value), pinhead:PINHD-2X6
- added JP2: JUMPER-SMT_2_NC_PASTE_NO-SILK, SparkFun-Jumpers:JUMPER-SMT_2_NC_PASTE_NO-SILK
- added R17: 68XR10KLF, 68XR10KLF:68XR10KLF
- added R20: (no value), rcl:R-US_R0603
- added R23, R24, R26, R33, R35: 10K, microbuilder:RESISTOR0603
- added R31, R32, R34: 1K, microbuilder:RESISTOR0603
- added U10: TLV6713DDCTDDC0006A_M, TLV6713DDC:TLV6713DDCTDDC0006A_M
- added U13: MCP1792T-5002H/CB, MCP1792T-5002H:MCP1792T-5002H/CB
- U4: value ADS1015IDGSR -> ADS1015IDGST; device ADS1015IDGSR:ADS1015IDGSR -> microbuilder:ADC_ADS1015
Connections:
- new net BATT_SENSE: R32.1, R33.2, U4.AIN0
- new net CHASSIS: JP2.1
- new net MOTOR_PULLUP: J9.1, R13.2
- new net M_N_GATE: U10.OUT
- new net N$27: R26.2, R31.1, U4.AIN1
- new net N$28: J2.1, J9.2
- new net N$29: R34.1, R35.2, U4.AIN2
- new net N$30: J3.1, J8.2
- new net N$9: R17.1, R20.1, U10.SENSE
- new net SCL: J10.2, R23.2, U4.SCL
- new net SDA: J10.1, R24.2, U4.SDA
- new net SYSTEM_PULLUP: J2.2, J8.1, R14.2
- net 5V: now also C39.P$2, J5.1, J6.1, JP1.1, JP1.3, R23.1, R24.1, U4.VDD
- net 5V_ALWAYS_ON: now also C37.1, J3.2, U10.VCC, U13.VOUT; no longer R13.2, R14.2
- net BATT_IN: now also R20.2, R33.1; no longer J2.2, J3.2, J8.2, J9.2
- net GND: now also C37.2, C38.2, C39.P$1, J1.2, J1.3, J4.2, J5.2, J6.2, J7.2, JP1.10, JP1.12, JP1.2, JP1.4, JP1.6, JP1.8, JP2.2, R17.2, R31.2, R32.2, R34.2, U10.GND, U13.GND, U4.ADDR, U4.GND
- net PS_IN: now also J1.1, R26.1
- net SYSTEM_IN: now also C38.1, U13.VIN
- net SYSTEM_SWITCHED: now also JP1.5, JP1.7
- net V_ADJ: now also J4.1, J7.1, JP1.11, JP1.9, R35.1
Other:
- note added: "Default I²C Address = 1001000"
- note added: "Motor Under Voltage"
- moved on the sheet: J2, J3, J4, J5, J6, J7, J8, J9

Commit message: Finished Routing PCB, Needs Design Review
Parts:
- removed R30: 1.62K, rcl:R-US_R0603
- removed U11: TLV7041DCKR, TLV7041DCKR:TLV7041DCKR
- removed U12: DMN67D8LW-13, DMN67D8LW-13:DMN67D8LW-13
- added LED4: (no value), led:LEDCHIP-LED0603
- added R36: 10K, microbuilder:RESISTOR0603
- added R37: 1K, microbuilder:RESISTOR0603
- R19: value 10K -> 1K
- R22: value 10K -> 5K
- R25: value (none) -> 2K
- R29: value 1.8K -> 2K
Connections:
- removed net N$3: R19.1, R29.2, U11.IN+
- removed net N_GATE: R14.1, R16.1, U6.G
- removed net N_GATE_M: R12.1, R13.1, U7.G
- removed net PS_SV_COMP: R25.1, U11.OUT, U12.G
- removed net ROBOT_V+: C17.1, C18.1, C19.1, C4.1, C5.1, C6.1
- removed net SYS_UV_SOURCE: U12.S, U9.OUT
- new net N$31: R36.2, R37.1, U4.AIN3
- new net N$32: LED3.A, R25.2
- new net N$33: LED2.A, R22.2
- new net N$34: LED1.A, R19.2
- net 5V: now also R19.1
- net 5V_ALWAYS_ON: no longer R25.2
- net BATT_IN: no longer R21.2, R22.2
- net GND: now also LED1.C, LED2.C, LED3.C, LED4.C, R37.2; no longer R29.1, R30.1
- net MOTOR_V+: now also R29.1, R36.1
- net M_N_GATE: now also R12.1, R13.1, U7.G
- net N$6: now also LED4.A, R29.2; no longer R22.1, R30.2, U11.IN-
- net PS_IN: no longer R19.2
- net SYSTEM_IN: now also R21.2, R25.1
- net SYSTEM_SWITCHED: now also C17.1, C18.1, C19.1, C4.1, C5.1, C6.1
- net S_N_GATE: now also R14.1, R16.1, U6.G, U9.OUT; no longer U12.D
- net V_ADJ: now also R22.1
Other:
- note added: "AMBER, 2.0v, 5mA"
- note added: "BLUE, 2.9v, 5mA"
- note added: "GREEN, 3.2V, 20mA"
- note added: "RED, 2.2v, 20mA"
- note removed: "This circuit ensures that the system under voltage only applies if power supply voltage is lower than battery voltage"
- moved on the sheet: LED1, LED2, LED3, R17, R18, R20, R21, R26, R31, R32, R33, R34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

Commit message: added UV 30s delay circuit
Parts:
- added C40, C41: 220uF, rcl:C-EUC1210
- added R30, R39: 1K, rcl:R-US_R0603
- added R38, R42: 62K, rcl:R-US_R0603
- added R40, R41: 100R, rcl:R-US_R0603
- added U11, U14: TLV6713DDCTDDC0006A_M, TLV6713DDC:TLV6713DDCTDDC0006A_M
- added U12, U5: DMN67D8LW-13, DMN67D8LW-13:DMN67D8LW-13
Connections:
- new net N$3: R30.1, U10.OUT, U5.G
- new net N$35: C40.1, R38.2, U11.SENSE, U5.S
- new net N$36: R40.1, U5.D
- new net N$37: R39.1, U12.G, U9.OUT
- new net N$38: R41.1, U12.D
- new net N$39: C41.1, R42.2, U12.S, U14.SENSE
- net 5V_ALWAYS_ON: now also R30.2, R39.2, R40.2, R41.2, U11.VCC, U14.VCC
- net GND: now also C40.2, C41.2, R38.1, R42.1, U11.GND, U14.GND
- net M_N_GATE: now also U11.OUT; no longer U10.OUT
- net S_N_GATE: now also U14.OUT; no longer U9.OUT
Other:
- note added: "30 Second Filter Circuit"
- note added: "Switch to a two stage approach where second stage has supercapacitor RC circuit"
- moved on the sheet: R18, R21

Commit message: Organized Schematic, Ready for Detailed Review
Parts:
- C7, C8: value 4.7uF -> 2.2uF
Other:
- note added: "(For Battery/Power Supply Hot-Swapping)"
- note added: "12v Switching Regulator"
- note added: "4 Channel I2C ADC"
- note added: "5v Switching Regulator"
- note added: "Always-on 5v Regulator"
- note added: "Bulk capacitance shown on the other Reg. circuit"
- note added: "Emergency Stop Ports"
- note added: "GND to Robot Chassis Jumper"
- note added: "Ideal Diode Circuits"
- note added: "Motor Power Ports"
- note added: "Power Expansion Port"
- note added: "Power Input"
- note added: "Power Outputs"
- note added: "Power Status LEDs"
- note added: "Power Supply Input"
- note added: "System Bulk Capacitance"
- note added: "Under- Voltage Protection Circuitry"
- note removed: "Check the R2 value !"
- note removed: "HOT SWAP INPUT"
- note removed: "POWER INPUT"
- note removed: "Switch to a two stage approach where second stage has supercapacitor RC circuit"
- moved on the sheet: C1, C2, C29, C3, C30, C31, C32, C33, C34, C35, C36, C37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
