File: Tello_Power_PCB_XT30_Extension.brd (EAGLE design)
At the start: 64 x 22.2 mm, 4 parts, among them CON1 XT30PW-F, CON2 XT30PW-F, CON3 XT30PW-F, CON4 XT30PW-F

Commit message: Added mfg files and renders
Connections:
- net + renamed V+
- net - renamed GND
Routing:
- net V+: track 0.00 -> 7.36 mm, vias 0 -> 1
- added copper zone on layer 16, net GND
- added copper zone on layer 1, net V+
Changed lines of the file:
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@@
 <text x="-2.8" y="18.2" size="2" layer="22" font="vector" ratio="15" rot="MR0">Motors</text>
 <text x="-16.8" y="18.2" size="2" layer="22" font="vector" ratio="15" rot="MR0">Motors</text>
-<wire x1="-26.5" y1="21.5" x2="-26.5" y2="16" width="0.1524" layer="22"/>
+<wire x1="-26.5" y1="19.5" x2="-26.5" y2="16" width="0.1524" layer="22"/>
 <wire x1="-26.5" y1="16" x2="-15.5" y2="16" width="0.1524" layer="22"/>
 <wire x1="-15.5" y1="16" x2="-15.5" y2="21.5" width="0.1524" layer="22"/>
@@
 <wire x1="15.5" y1="21.5" x2="15.5" y2="16" width="0.1524" layer="22"/>
 <wire x1="15.5" y1="16" x2="26.5" y2="16" width="0.1524" layer="22"/>
-<wire x1="26.5" y1="16" x2="26.5" y2="21.5" width="0.1524" layer="22"/>
+<wire x1="26.5" y1="16" x2="26.5" y2="19.5" width="0.1524" layer="22"/>
 <hole x="-29" y="9" drill="2.7"/>
 <circle x="-29" y="9" radius="2.5" width="0.1" layer="21"/>
@@
 </elements>
 <signals>
-<signal name="+">
+<signal name="GND">
+<contactref element="CON1" pad="-"/>
+<contactref element="CON4" pad="-"/>
+<contactref element="CON3" pad="-"/>
+<contactref element="CON2" pad="-"/>
+<via x="29" y="9" extent="1-16" drill="2.7" diameter="5"/>
+<polygon width="1" layer="16" isolate="0.254" thermals="no">
+<vertex x="-33" y="23"/>
+<vertex x="34" y="23"/>
+<vertex x="34" y="-1"/>
+<vertex x="-33" y="-1"/>
+</polygon>
+</signal>
+<signal name="V+">
 <contactref element="CON1" pad="+"/>
 <contactref element="CON2" pad="+"/>
 <contactref element="CON3" pad="+"/>
 <contactref element="CON4" pad="+"/>
-<wire x1="9.5" y1="7.5" x2="23.5" y2="7.5" width="0" layer="19" extent="1-1"/>
-<wire x1="-4.5" y1="7.5" x2="9.5" y2="7.5" width="0" layer="19" extent="1-1"/>
-<wire x1="-18.5" y1="7.5" x2="-4.5" y2="7.5" width="0" layer="19" extent="1-1"/>
-</signal>
-<signal name="-">
-<contactref element="CON1" pad="-"/>
-<contactref element="CON2" pad="-"/>
-<contactref element="CON3" pad="-"/>
-<contactref element="CON4" pad="-"/>
-<wire x1="4.5" y1="7.5" x2="18.5" y2="7.5" width="0" layer="19" extent="1-1"/>
-<wire x1="-9.5" y1="7.5" x2="4.5" y2="7.5" width="0" layer="19" extent="1-1"/>
-<wire x1="-23.5" y1="7.5" x2="-9.5" y2="7.5" width="0" layer="19" extent="1-1"/>
-</signal>
-<signal name="N$6">
-<via x="29" y="9" extent="1-16" drill="2.7" diameter="5"/>
-</signal>
-<signal name="N$8">
 <via x="29" y="3" extent="1-16" drill="2.7" diameter="5"/>
+<wire x1="29" y1="3" x2="24.5" y2="7.5" width="2.54" layer="1"/>
+<wire x1="24.5" y1="7.5" x2="23.5" y2="7.5" width="2.54" layer="1"/>
+<polygon width="1" layer="1" isolate="0.254" thermals="no">
+<vertex x="34" y="23"/>
+<vertex x="34" y="23"/>
+<vertex x="34" y="-1"/>
+<vertex x="-33" y="-1"/>
+<vertex x="-33" y="23"/>
+</polygon>
 </signal>
 </signals>
