File: Tello_Power_PCB_XT30_Extension.sch (EAGLE design)
At the start: 4 parts, among them CON1 XT30PW-F, CON2 XT30PW-F, CON3 XT30PW-F, CON4 XT30PW-F

Commit message: Added mfg files and renders
Connections:
- new net GND: CON1.-, CON2.-, CON3.-, CON4.-
- new net V+: CON1.+, CON2.+, CON3.+, CON4.+
