File: Tello_Power_PCB.brd (EAGLE design)
At the start: 122.5 x 89.3 mm, 134 parts, among them CON1 XT30PW-F, CON2 XT30PW-F, CON3 XT30PW-F, CON4 XT30PW-F, CON7 XT60PW-M, J1 PJ-002A, J10 SM02BGHSTBLFSN, J2 1719740002, J3 1719740002, J4 1719740002, J5 1719740002, J6 1719740002, J7 1719740002, J8 1719740002, J9 1719740002, M1 30V, M2 60V, M3 30V, M4 60V, Q1 BSC027N06LS5ATMA1, Q2 BSC027N06LS5ATMA1, Q3 IXTA96P085T, Q7 IXTA96P085T, Q8 IXTA96P085T, Q9 IXTA96P085T, U1 LM3150MH/NOPB, U10 TLV6713DDCTDDC0006A_M, U11 TLV6713DDCTDDC0006A_M, U12 DMN67D8LW-13, U13 MCP1792T-5002H/CB, U14 TLV6713DDCTDDC0006A_M, U2 LM3150MH/NOPB, U3 LTC4357CMS8TRPBF, U4 ADS1015IDGST, U5 DMN67D8LW-13, U6 DMN67D8LW-13, U7 DMN67D8LW-13, U8 LTC4357CMS8TRPBF, U9 TLV6713DDCTDDC0006A_M

Commit message: Organized Schematic
Parts:
- R20, R21: value (none) -> 100K
Changed lines of the file:
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@@
 <attribute name="NAME" x="27.82" y="-18.93" size="0.4064" layer="27" font="vector" ratio="6" rot="SR180"/>
 </element>
-<element name="R21" library="rcl" library_urn="urn:adsk.eagle:library:334" package="R0603" package3d_urn="urn:adsk.eagle:package:23555/3" value="" x="21.26" y="-48.91" smashed="yes">
+<element name="R21" library="rcl" library_urn="urn:adsk.eagle:library:334" package="R0603" package3d_urn="urn:adsk.eagle:package:23555/3" value="100K" x="21.26" y="-48.91" smashed="yes">
 <attribute name="NAME" x="20.625" y="-48.275" size="0.6" layer="25"/>
 <attribute name="POPULARITY" value="77" x="21.26" y="-48.91" size="1.778" layer="27" font="vector" display="off"/>
@@
 <attribute name="NAME" x="-15.5908" y="-4.2888" size="1.27" layer="27" ratio="6" rot="SR270"/>
 </element>
-<element name="R20" library="rcl" library_urn="urn:adsk.eagle:library:334" package="R0603" package3d_urn="urn:adsk.eagle:package:23555/3" value="" x="25.79" y="-30.41" smashed="yes">
+<element name="R20" library="rcl" library_urn="urn:adsk.eagle:library:334" package="R0603" package3d_urn="urn:adsk.eagle:package:23555/3" value="100K" x="25.79" y="-30.41" smashed="yes">
 <attribute name="NAME" x="24.525" y="-29.635" size="0.6096" layer="25"/>
 <attribute name="POPULARITY" value="77" x="-1.21" y="-30.41" size="0.4064" layer="27" display="off"/>

Commit message: Added mfg files and renders
Parts:
- C1, C2, C29, C36, C38: device rcl:C1206 -> Tello_Power_PCB:RCL_C1206
- C10, C13, C15, C9, R2, R3: device 12v- LM3150:0805 -> Tello_Power_PCB:12V--LM3150_0805:1
- C11, R1: device 12v- LM3150:0402 -> Tello_Power_PCB:12V--LM3150_0402
- C12, C24: device CGA4F2C0G1H153J085AA:CAPC2012X100N -> Tello_Power_PCB:CGA4F2C0G1H153J085AA_CAPC2012X100N
- C14: device 12v- LM3150:1206 -> Tello_Power_PCB:12V--LM3150_1206:1
- C16: device 12v- LM3150:PCV1E330MCL1GS -> Tello_Power_PCB:12V--LM3150_PCV1E330MCL1GS
- C17, C18, C19, C4, C5, C6: value PCR1H820MCL1GS -> PCR1H820MCL1GS_PCR1H820MCL1GS; device PCR1H820MCL1GS:CAP_PC_10X8_NCH -> Tello_Power_PCB:PCR1H820MCL1GS_CAP_PC_10X8_NCH
- C20: device 5v-LM3150MH:6032-28 -> Tello_Power_PCB:5V-LM3150MH_6032-28
- C21, C22, C25, C27, R10, R7, R8, R9: device 5v-LM3150MH:0805 -> Tello_Power_PCB:5V-LM3150MH_0805
- C23, R6: device 5v-LM3150MH:0603 -> Tello_Power_PCB:5V-LM3150MH_0603
- C26: device 5v-LM3150MH:1206 -> Tello_Power_PCB:5V-LM3150MH_1206
- C28: device 5v-LM3150MH:C2917 -> Tello_Power_PCB:5V-LM3150MH_C2917
- C3, C30, C37: device rcl:C0603 -> Tello_Power_PCB:RCL_C0603
- C31, C32, C33, C34, C35: value 227AVG050MGBJ -> 227AVG050MGBJ_227AVG050MGBJ; device 227AVG050MGBJ:CAPPRD500W60D1025H1350 -> Tello_Power_PCB:227AVG050MGBJ_CAPPRD500W60D1025H1350
- C39, R23, R24, R26, R31, R32, R33, R34, R35, R36, R37: device microbuilder:0603 -> Tello_Power_PCB:MICROBUILDER_0603:1
- C40, C41: device rcl:C1210 -> Tello_Power_PCB:RCL_C1210
- C7, C8: device 12v- LM3150:3528-21 -> Tello_Power_PCB:12V--LM3150_3528-21
- CON1, CON2, CON3, CON4: value XT30PW-F -> AMASS_XT30PW-F; device amass:XT30PW-F -> Tello_Power_PCB:AMASS_XT30PW-F
- CON7: value XT60PW-M -> AMASS_XT60PW-M; device amass:XT60PW-M -> Tello_Power_PCB:AMASS_XT60PW-M
- CR1, CR2: value STPS1150A -> STPS1150A_STPS1150A; device STPS1150A:SMA_STM -> Tello_Power_PCB:STPS1150A_SMA_STM
- J1: value PJ-002A -> PJ-002A_PJ-002A; device PJ-002A:CUI_PJ-002A -> Tello_Power_PCB:PJ-002A_CUI_PJ-002A
- J10: value SM02BGHSTBLFSN -> SM02B-GHS-TB_SM02BGHSTBLFSN; device SM02B-GHS-TB:CONN_SM02BGHSTB_JST -> Tello_Power_PCB:SM02B-GHS-TB_CONN_SM02BGHSTB_JST
- J2, J3, J4, J5, J6, J7, J8, J9: value 1719740002 -> 1719740002_1719740002; device 1719740002:MOLEX_1719740002 -> Tello_Power_PCB:1719740002_MOLEX_1719740002
- JP1: device pinhead:2X06 -> Tello_Power_PCB:PINHEAD_2X06
- JP2: value JUMPER-SMT_2_NC_PASTE_NO-SILK -> SPARKFUN-JUMPERS_JUMPER-SMT_2_NC_PASTE_NO-SILK; device SparkFun-Jumpers:SMT-JUMPER_2_NC_PASTE_NO-SILK -> Tello_Power_PCB:SPARKFUN-JUMPERS_SMT-JUMPER_2_NC_PASTE_NO-SILK
- L1: device 12v- LM3150:WE-LHMI_8040 -> Tello_Power_PCB:12V--LM3150_WE-LHMI_8040
- L2: device 5v-LM3150MH:XAL5030 -> Tello_Power_PCB:5V-LM3150MH_XAL5030
- L3: device XAL4030-332MEB:XAL4030-332MEB -> Tello_Power_PCB:XAL4030-332MEB_XAL4030-332MEB
- L4: device 5v-LM3150MH:IND_NPI43C -> Tello_Power_PCB:5V-LM3150MH_IND_NPI43C
- LED1, LED2, LED3, LED4: device led:CHIP-LED0603 -> Tello_Power_PCB:LED_CHIP-LED0603
- M1, M2: device 12v- LM3150:TRANS_NEXFET_Q5A -> Tello_Power_PCB:12V--LM3150_TRANS_NEXFET_Q5A:1
- M3, M4: device 5v-LM3150MH:TRANS_NEXFET_Q5A -> Tello_Power_PCB:5V-LM3150MH_TRANS_NEXFET_Q5A
- Q1, Q2: value BSC027N06LS5ATMA1 -> BSC027N06LS5ATMA1_BSC027N06LS5ATMA1; device BSC027N06LS5ATMA1:BSC027N06LS5ATMA1 -> Tello_Power_PCB:BSC027N06LS5ATMA1_BSC027N06LS5ATMA1
- Q3, Q7, Q8, Q9: value IXTA96P085T -> IXTA96P085T_IXTA96P085T; device IXTA96P085T:IXTA96P085T -> Tello_Power_PCB:IXTA96P085T_IXTA96P085T
- R11: device rcl:R0805 -> Tello_Power_PCB:RCL_R0805
- R12, R13, R14, R15, R16, R19, R20, R21, R22, R25, R27, R28, R29, R30, R38, R39, R40, R41, R42, R5: device rcl:R0603 -> Tello_Power_PCB:RCL_R0603
- R17, R18, R4: value 68XR10KLF -> 68XR10KLF_68XR10KLF; device 68XR10KLF:RES3_68X_TTE -> Tello_Power_PCB:68XR10KLF_RES3_68X_TTE
- U1, U2: value LM3150MH/NOPB -> 5V-LM3150MH_LM3150MH/NOPB; device 5v-LM3150MH:MXA14A -> Tello_Power_PCB:5V-LM3150MH_MXA14A
- U10, U11, U14, U9: value TLV6713DDCTDDC0006A_M -> TLV6713DDC_TLV6713DDCTDDC0006A_M; device TLV6713DDC:DDC0006A_M -> Tello_Power_PCB:TLV6713DDC_DDC0006A_M
- U12, U5, U6, U7: value DMN67D8LW-13 -> DMN67D8LW-13_DMN67D8LW-13; device DMN67D8LW-13:DMN67D8LW-13_DIO -> Tello_Power_PCB:DMN67D8LW-13_DMN67D8LW-13_DIO
- U13: value MCP1792T-5002H/CB -> MCP1792T-5002H_MCP1792T-5002H/CB; device MCP1792T-5002H:SOT-23A_CB_MCH -> Tello_Power_PCB:MCP1792T-5002H_SOT-23A_CB_MCH
- U3, U8: value LTC4357CMS8TRPBF -> LTC4357_LTC4357CMS8TRPBF; device LTC4357:MSOP-8_MS_LIT -> Tello_Power_PCB:LTC4357_MSOP-8_MS_LIT
- U4: device microbuilder:MSOP10 -> Tello_Power_PCB:MICROBUILDER_MSOP10

Commit message: updated readme photos
Parts:
- R15, R5: value 10K -> 100R
Changed lines of the file:
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@@
 <attribute name="SPICEPREFIX" value="R" x="15.05" y="-44.23" size="1.778" layer="27" rot="R180" display="off"/>
 </element>
-<element name="R15" library="Tello_Power_PCB" library_urn="urn:adsk.eagle:library:37573195" package="RCL_R0603" package3d_urn="urn:adsk.eagle:package:37573323/1" value="10K" x="11.46" y="-43.35" smashed="yes" rot="R180">
+<element name="R15" library="Tello_Power_PCB" library_urn="urn:adsk.eagle:library:37573195" package="RCL_R0603" package3d_urn="urn:adsk.eagle:package:37573323/1" value="100R" x="11.46" y="-43.35" smashed="yes" rot="R180">
 <attribute name="NAME" x="12.095" y="-43.985" size="0.4064" layer="25" font="vector" rot="R180"/>
 <attribute name="POPULARITY" value="77" x="11.46" y="-43.35" size="1.778" layer="27" rot="R180" display="off"/>
@@
 <attribute name="SPICEPREFIX" value="C" x="25.98" y="-19.32" size="1.778" layer="27" display="off"/>
 </element>
-<element name="R5" library="Tello_Power_PCB" library_urn="urn:adsk.eagle:library:37573195" package="RCL_R0603" package3d_urn="urn:adsk.eagle:package:37573323/1" value="10K" x="25.98" y="-20.98" smashed="yes">
+<element name="R5" library="Tello_Power_PCB" library_urn="urn:adsk.eagle:library:37573195" package="RCL_R0603" package3d_urn="urn:adsk.eagle:package:37573323/1" value="100R" x="25.98" y="-20.98" smashed="yes">
 <attribute name="NAME" x="27.78" y="-21.24" size="0.4064" layer="25" font="vector" rot="R90"/>
 <attribute name="POPULARITY" value="77" x="25.98" y="-20.98" size="1.778" layer="27" display="off"/>

Commit message: updated high side switch resistors
Parts:
- R12, R16: value 10K -> 2K
- R15, R5: value 100R -> 3.6K
Changed lines of the file:
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@@
 <attribute name="SPICEPREFIX" value="R" x="15.05" y="-44.23" size="1.778" layer="27" rot="R180" display="off"/>
 </element>
-<element name="R15" library="Tello_Power_PCB" library_urn="urn:adsk.eagle:library:37573195" package="RCL_R0603" package3d_urn="urn:adsk.eagle:package:37573323/1" value="100R" x="11.46" y="-43.35" smashed="yes" rot="R180">
+<element name="R15" library="Tello_Power_PCB" library_urn="urn:adsk.eagle:library:37573195" package="RCL_R0603" package3d_urn="urn:adsk.eagle:package:37573323/1" value="3.6K" x="11.46" y="-43.35" smashed="yes" rot="R180">
 <attribute name="NAME" x="12.095" y="-43.985" size="0.4064" layer="25" font="vector" rot="R180"/>
 <attribute name="POPULARITY" value="77" x="11.46" y="-43.35" size="1.778" layer="27" rot="R180" display="off"/>
 <attribute name="SPICEPREFIX" value="R" x="11.46" y="-43.35" size="1.778" layer="27" rot="R180" display="off"/>
 </element>
-<element name="R16" library="Tello_Power_PCB" library_urn="urn:adsk.eagle:library:37573195" package="RCL_R0603" package3d_urn="urn:adsk.eagle:package:37573323/1" value="10K" x="15.05" y="-46.2" smashed="yes">
+<element name="R16" library="Tello_Power_PCB" library_urn="urn:adsk.eagle:library:37573195" package="RCL_R0603" package3d_urn="urn:adsk.eagle:package:37573323/1" value="2K" x="15.05" y="-46.2" smashed="yes">
 <attribute name="NAME" x="14.565" y="-45.455" size="0.4064" layer="25" font="vector"/>
 <attribute name="POPULARITY" value="77" x="15.05" y="-46.2" size="1.778" layer="27" display="off"/>
@@
 <attribute name="SPICEPREFIX" value="R" x="55.98" y="-17.65" size="1.778" layer="27" rot="R180" display="off"/>
 </element>
-<element name="R12" library="Tello_Power_PCB" library_urn="urn:adsk.eagle:library:37573195" package="RCL_R0603" package3d_urn="urn:adsk.eagle:package:37573323/1" value="10K" x="25.78" y="-26.08" smashed="yes">
+<element name="R12" library="Tello_Power_PCB" library_urn="urn:adsk.eagle:library:37573195" package="RCL_R0603" package3d_urn="urn:adsk.eagle:package:37573323/1" value="2K" x="25.78" y="-26.08" smashed="yes">
 <attribute name="NAME" x="27.33" y="-25.66" size="0.4064" layer="25" font="vector" rot="R270"/>
 <attribute name="POPULARITY" value="77" x="20.78" y="-21.08" size="1.778" layer="27" display="off"/>
@@
 <attribute name="SPICEPREFIX" value="C" x="25.98" y="-19.32" size="1.778" layer="27" display="off"/>
 </element>
-<element name="R5" library="Tello_Power_PCB" library_urn="urn:adsk.eagle:library:37573195" package="RCL_R0603" package3d_urn="urn:adsk.eagle:package:37573323/1" value="100R" x="25.98" y="-20.98" smashed="yes">
+<element name="R5" library="Tello_Power_PCB" library_urn="urn:adsk.eagle:library:37573195" package="RCL_R0603" package3d_urn="urn:adsk.eagle:package:37573323/1" value="3.6K" x="25.98" y="-20.98" smashed="yes">
 <attribute name="NAME" x="27.78" y="-21.24" size="0.4064" layer="25" font="vector" rot="R90"/>
 <attribute name="POPULARITY" value="77" x="25.98" y="-20.98" size="1.778" layer="27" display="off"/>
